File: RP-006440-DD-2-RP2350A Minimal Board Kicad/RP2350_60QFN_minimal.kicad_sch (KiCad schematic)
At the start: 43 parts, among them J1 USB_B_Micro, J2 Conn_02x18_Odd_Even, J3 Conn_02x18_Odd_Even, J4 SM03B-SRSS-TB, SW1 SW_Push, SW2 SW_Push, U1 RP2350_60QFN, U2 NCP1117-3.3_SOT223, U3 W25Q128JVS, Y1 ABM8-272-T3

Commit message: Updated with USB-C circuit for review
Parts:
- added C20, C21: 100nF, Capacitor_SMD:C_0402_1005Metric, symbol Device:C
- added C22, C23: 10nF, Capacitor_SMD:C_0402_1005Metric, symbol Device:C
- added R11, R3: 5.1K, Resistor_SMD:R_0402_1005Metric, symbol Device:R
- added R12, R13: 27, Resistor_SMD:R_0402_1005Metric, symbol Device:R
- added U4: AMS1117-3.3, Package_TO_SOT_SMD:SOT-223-3_TabPin2, symbol Regulator_Linear:AMS1117-3.3
- added USB1: TYPE-C 16PIN 2MD(073), C2765186-usbc:USB-C-SMD_TYPE-C-6PIN-2MD-073, symbol C2765186-usbc:TYPE-C16PIN2MD(073)
Connections:
- net +3V3: now also C21.1, C23.1, U4.2 (VO)
- net GND: now also C20.2, C21.2, C22.2, C23.2, R11.2, R3.2, U4.1 (GND), USB1.1 (GND), USB1.12 (GND), USB1.13 (SHELL), USB1.14 (SHELL)
- net USB_D+: now also R12.2
- net USB_D-: now also R13.2
- net VBUS: now also C20.1, C22.1, U4.3 (VI), USB1.11 (VBUS), USB1.2 (VBUS)
- new net: R11.1, USB1.10 (CC2)
- new net: R3.1, USB1.4 (CC1)
- new net USB2_D+: R12.1, USB1.6 (DP1), USB1.8 (DP2)
- new net USB2_D-: R13.1, USB1.5 (DN2), USB1.7 (DN1)
- no-connect marks 1 -> 3
Other:
- note added: "DO NOT USE. UNTESTED"
- note added: "Help? Do I need a diod here? what kind?"
- note added: "Help? What do I connect USB2_D -/+ to?"
- note added: "Power (Original/Old)"
- note added: "Power USB-C (New)"
- note added: "RP2350"
- note removed: "Power"
- company: Raspberry Pi Ltd -> Abluestar.com
- title: RP2350A QFN-60 Minimal Design Example -> RP2350A QFN-60 Minimal Design Example With USBC
- moved on the sheet: C10, C11, C12, C13, C14, C15, C16, C17, C18, C19, C2, C3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
